File: kicad/test.kicad_sch (KiCad schematic)
At the start: 0 parts

Commit message: 更新 README, 和 kicad-libs 封装测试工程
Parts:
- added C1, C10, C7, C9: 106, Capacitor_SMD:C_0805_2012Metric_Pad1.18x1.45mm_HandSolder, symbol Device:C_Small
- added C11, C2, C3, C6, C8: 104, Capacitor_SMD:C_0805_2012Metric_Pad1.18x1.45mm_HandSolder, symbol Device:C_Small
- added C4, C5: 100pF, Capacitor_SMD:C_0805_2012Metric_Pad1.18x1.45mm_HandSolder, symbol Device:C_Small
- added D1: SS34, Diode_SMD:D_SMA, symbol Diode:SS34
- added D2: LED, LED_SMD:LED_0805_2012Metric_Pad1.15x1.40mm_HandSolder, symbol Device:LED
- added J1: Header, Connector_PinSocket_2.54mm:PinSocket_1x04_P2.54mm_Vertical, symbol Connector_Generic:Conn_01x04
- added J2, J3, J4, J5: T, MountingHole:MountingHole_3.2mm_M3_DIN965_Pad, symbol Connector_Generic:Conn_01x01
- added R1, R6, R7: 1002, Resistor_SMD:R_0805_2012Metric_Pad1.20x1.40mm_HandSolder, symbol Device:R_Small
- added R10: 1000, Resistor_SMD:R_0805_2012Metric_Pad1.20x1.40mm_HandSolder, symbol Device:R_Small
- added R12: 5601, Resistor_SMD:R_0805_2012Metric_Pad1.20x1.40mm_HandSolder, symbol Device:R_Small
- added R13: 8201, Resistor_SMD:R_0805_2012Metric_Pad1.20x1.40mm_HandSolder, symbol Device:R_Small
- added R14: 51R, Resistor_SMD:R_0805_2012Metric_Pad1.20x1.40mm_HandSolder, symbol Device:R_Small
- added R2, R3: 1003, Resistor_SMD:R_0805_2012Metric_Pad1.20x1.40mm_HandSolder, symbol Device:R_Small
- added R4, R5: 4703, Resistor_SMD:R_0805_2012Metric_Pad1.20x1.40mm_HandSolder, symbol Device:R_Small
- added R8, R9: 4701, Resistor_SMD:R_0805_2012Metric_Pad1.20x1.40mm_HandSolder, symbol Device:R_Small
- added TH1: PT100, Connector_PinSocket_2.54mm:PinSocket_1x03_P2.54mm_Vertical, symbol Device:Thermistor_PTC_3Wire
- added TP1, TP2, TP3, TP4, TP5, TP6, TP7, TP8: TP, Connector_PinSocket_2.54mm:PinSocket_1x01_P2.54mm_Vertical, symbol Connector:TestPoint
- added U1: LM358, Package_SO:SOP-8_3.76x4.96mm_P1.27mm, symbol Amplifier_Operational:LM358
- added U3: TL431DBZ, Package_TO_SOT_SMD:SOT-23, symbol Reference_Voltage:TL431DBZ
Connections:
- new net: C4.1, R4.1, R6.2, TP3.1, U1.2 (-)
- new net: C4.2, R2.1, R4.2, TP2.1, U1.1
- new net: C5.2, R5.2, R7.2, TP4.1, U1.3 (+)
- new net: C3.2, R1.1, U1.6 (-), U1.7
- new net: C1.1, J1.2 (Pin_2), R1.2, TP1.1
- new net: R10.2, R6.1, R8.1, TP5.1
- new net: C2.1, R3.2, U1.5 (+)
- new net: R10.1, TH1.2
- new net: C3.1, R2.2, R3.1
- new net: C8.2, R12.1, R13.2, U3.1 (REF)
- new net: D1.2 (A), J1.1 (Pin_1)
- new net: R7.1, R9.1, TH1.1, TP6.1
- new net +4.2V: C6.2, C7.2, D2.2 (A), R12.2, R14.1, R8.2, R9.2, TP7.1, U3.2 (K)
- new net +5V: C10.1, C11.1, C9.2, D1.1 (K), R14.2, U1.8 (V+)
- new net GND: C1.2, C10.2, C11.2, C2.2, C5.1, C6.1, C7.1, C8.1, C9.1, D2.1 (K), J1.4 (Pin_4), J2.1 (Pin_1), J3.1 (Pin_1), J4.1 (Pin_1), J5.1 (Pin_1), R13.1, R5.1, TH1.3, TP8.1, U1.4 (V-), U3.3 (A)
- no-connect marks 0 -> 1
Other:
- note added: "PT100 ºãÑ¹µçÇÅµ÷ÀíµçÂ·"
- note added: "V1.0.0"

Commit message: 新增 LED 驱动芯片(包含LED5000,AL8860,TPS92365)库
Parts:
- added R11: 500R, Resistor_SMD:R_0805_2012Metric_Pad1.20x1.40mm_HandSolder, symbol Device:R_Small
Connections:
- net +4.2V: now also R11.2; no longer D2.2 (A)
- new net: D2.2 (A), R11.1
Other:
- note removed: "PT100 ºãÑ¹µçÇÅµ÷ÀíµçÂ·"
- moved on the sheet: D2
Changed lines of the file:
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@@
 		)
 	)
-	(text "PT100 ºãÑ¹µçÇÅµ÷ÀíµçÂ·"
+	(text ""
 		(exclude_from_sim no)
 		(at 213.868 170.18 0)
@@
 	(wire
 		(pts
-			(xy 130.81 125.73) (xy 130.81 130.81)
+			(xy 130.81 125.73) (xy 130.81 128.27)
 		)
 		(stroke
@@
 	(wire
 		(pts
-			(xy 130.81 146.05) (xy 130.81 138.43)
+			(xy 130.81 146.05) (xy 130.81 142.24)
 		)
 		(stroke
@@
 	(wire
 		(pts
+			(xy 130.81 133.35) (xy 130.81 134.62)
+		)
+		(stroke
+			(width 0)
+			(type default)
+		)
+	)
+	(wire
+		(pts
 			(xy 137.16 85.09) (xy 137.16 91.44)
 		)
@@
 	(symbol
 		(lib_id "Device:LED")
-		(at 130.81 134.62 90)
+		(at 130.81 138.43 90)
 		(unit 1)
 		(exclude_from_sim no)
@@
 		(dnp no)
 		(property "Reference" "D2"
-			(at 133.35 133.858 90)
+			(at 133.35 137.668 90)
 			(effects
 				(font
@@
 		)
 		(property "Value" "LED"
-			(at 133.096 135.5726 90)
+			(at 133.096 139.3826 90)
 			(effects
 				(font
@@
 		)
 		(property "Footprint" "LED_SMD:LED_0805_2012Metric_Pad1.15x1.40mm_HandSolder"
-			(at 130.81 134.62 0)
+			(at 130.81 138.43 0)
 			(effects
 				(font
@@
 		)
 		(property "Datasheet" "~"
-			(at 130.81 134.62 0)
+			(at 130.81 138.43 0)
 			(effects
 				(font
@@
 		)
 		(property "Description" "Light emitting diode"
-			(at 130.81 134.62 0)
+			(at 130.81 138.43 0)
 			(effects
 				(font
@@
 		)
 		(property "Sim.Pins" "1=K 2=A"
-			(at 130.81 134.62 0)
+			(at 130.81 138.43 0)
 			(effects
 				(font
@@
 					(unit 1)
 				)
+			)
+		)
+	)
+	(symbol
+		(lib_id "Device:R_Small")
+		(at 130.81 130.81 180)
+		(unit 1)
+		(exclude_from_sim no)
+		(in_bom yes)
+		(on_board yes)
+		(dnp no)
+		(property "Reference" "R11"
+			(at 134.62 130.302 0)
+			(effects
+				(font
+					(size 1.016 1.016)
+				)
+			)
+		)
+		(property "Value" "500R"
+			(at 134.62 131.826 0)
+			(effects
+				(font
+					(size 1.27 1.27)
+				)
+			)
+		)
+		(property "Footprint" "Resistor_SMD:R_0805_2012Metric_Pad1.20x1.40mm_HandSolder"
+			(at 130.81 130.81 0)
+			(effects
+				(font
+					(size 1.27 1.27)
+				)
+				(hide yes)
+			)
+		)
+		(property "Datasheet" "~"
+			(at 130.81 130.81 0)
+			(effects
+				(font
+					(size 1.27 1.27)
+				)
+				(hide yes)
+			)
+		)
+		(property "Description" "Resistor, small symbol"
+			(at 130.81 130.81 0)
+			(effects
+				(font
+					(size 1.27 1.27)
+				)
+				(hide yes)
+			)
+		)
+		(pin "2"
+		)
+		(pin "1"
+		)
+		(instances
+			(project "test"
+				(path "/46f61707-7257-4955-981c-56313ea3fc5c"
+					(reference "R11")
+					(unit 1)
+				)
